Commit message: Add: Meshes

File: urdf/omnibot.urdf.xacro (robot description, xacro)
@@ -5,5 +5,5 @@
     <visual>
       <geometry>
-        <box size="0.3 0.3 0.1"/>
+        <mesh filename="package://omnibot_description/meshes/base.stl" scale="1 1 1"/>
       </geometry>
       <material name="blue">
@@ -13,5 +13,5 @@
     <collision>
       <geometry>
-        <box size="0.3 0.3 0.1"/>
+        <mesh filename="package://omnibot_description/meshes/base.stl" scale="1 1 1"/>
       </geometry>
     </collision>
@@ -21,10 +21,10 @@
     </inertial>
   </link>
-  <!-- 4 Mecanum wheels (simplified as cylinders) -->
+  <!-- 4 Mecanum wheels using mesh -->
   <xacro:macro name="wheel" params="name x y">
     <link name="${name}">
       <visual>
         <geometry>
-          <cylinder radius="0.04" length="0.02"/>
+          <mesh filename="package://omnibot_description/meshes/wheel.stl" scale="1 1 1"/>
         </geometry>
         <material name="black">
@@ -34,5 +34,5 @@
       <collision>
         <geometry>
-          <cylinder radius="0.04" length="0.02"/>
+          <mesh filename="package://omnibot_description/meshes/wheel.stl" scale="1 1 1"/>
         </geometry>
       </collision>

Commit message: urdf

File: urdf/omnibot.urdf.xacro (robot description, xacro)
@@ -1,5 +1,5 @@
 <?xml version="1.0"?>
 <robot xmlns:xacro="http://www.ros.org/wiki/xacro" name="omnibot">
-  <!-- Base link -->
+  <!-- ================= Base Link ================= -->
   <link name="base_link">
     <visual>
@@ -7,4 +7,6 @@
         <mesh filename="package://omnibot_description/meshes/base.stl" scale="1 1 1"/>
       </geometry>
+      <!-- Base-Mesh auf Rädern platzieren -->
+      <origin xyz="0 0 0.09" rpy="0 0 0"/>
       <material name="blue">
         <color rgba="0.1 0.1 0.8 1"/>
@@ -15,4 +17,5 @@
         <mesh filename="package://omnibot_description/meshes/base.stl" scale="1 1 1"/>
       </geometry>
+      <origin xyz="0 0 0.09" rpy="0 0 0"/>
     </collision>
     <inertial>
@@ -21,6 +24,6 @@
     </inertial>
   </link>
-  <!-- 4 Mecanum wheels using mesh -->
-  <xacro:macro name="wheel" params="name x y">
+  <!-- ================= Wheel Macro ================= -->
+  <xacro:macro name="wheel" params="name x y rpy_r rpy_p rpy_y">
     <link name="${name}">
       <visual>
@@ -28,4 +31,6 @@
           <mesh filename="package://omnibot_description/meshes/wheel.stl" scale="1 1 1"/>
         </geometry>
+        <!-- Z = H_wheel/2 -->
+        <origin xyz="0 0 0.04" rpy="0 0 0"/>
         <material name="black">
           <color rgba="0.02 0.02 0.02 1"/>
@@ -36,4 +41,5 @@
           <mesh filename="package://omnibot_description/meshes/wheel.stl" scale="1 1 1"/>
         </geometry>
+        <origin xyz="0 0 0.04" rpy="0 0 0"/>
       </collision>
       <inertial>
@@ -45,11 +51,13 @@
       <parent link="base_link"/>
       <child link="${name}"/>
-      <origin xyz="${x} ${y} -0.05" rpy="0 1.5708 0"/>
+      <!-- Position relativ zum base_link -->
+      <origin xyz="${x} ${y} 0" rpy="${rpy_r} ${rpy_p} ${rpy_y}"/>
       <axis xyz="0 1 0"/>
     </joint>
   </xacro:macro>
-  <xacro:wheel name="wheel_fl" x="0.12" y="0.12"/>
-  <xacro:wheel name="wheel_fr" x="0.12" y="-0.12"/>
-  <xacro:wheel name="wheel_rl" x="-0.12" y="0.12"/>
-  <xacro:wheel name="wheel_rr" x="-0.12" y="-0.12"/>
+  <!-- ================= Four Mecanum Wheels ================= -->
+  <xacro:wheel name="wheel_fl" x="0.12" y="0.12" rpy_r="0" rpy_p="0" rpy_y="0"/>
+  <xacro:wheel name="wheel_fr" x="0.12" y="-0.12" rpy_r="0" rpy_p="0" rpy_y="0"/>
+  <xacro:wheel name="wheel_rl" x="-0.12" y="0.12" rpy_r="0" rpy_p="0" rpy_y="0"/>
+  <xacro:wheel name="wheel_rr" x="-0.12" y="-0.12" rpy_r="0" rpy_p="0" rpy_y="0"/>
 </robot>

Commit message: Fix: Joints Wheels

File: urdf/omnibot.urdf.xacro (robot description, xacro)
@@ -7,6 +7,5 @@
         <mesh filename="package://omnibot_description/meshes/base.stl" scale="1 1 1"/>
       </geometry>
-      <!-- Base-Mesh auf Rädern platzieren -->
-      <origin xyz="0 0 0.09" rpy="0 0 0"/>
+      <origin xyz="0 0 0" rpy="0 0 0"/>
       <material name="blue">
         <color rgba="0.1 0.1 0.8 1"/>
@@ -17,5 +16,5 @@
         <mesh filename="package://omnibot_description/meshes/base.stl" scale="1 1 1"/>
       </geometry>
-      <origin xyz="0 0 0.09" rpy="0 0 0"/>
+      <origin xyz="0 0 0" rpy="0 0 0"/>
     </collision>
     <inertial>
@@ -24,40 +23,116 @@
     </inertial>
   </link>
-  <!-- ================= Wheel Macro ================= -->
-  <xacro:macro name="wheel" params="name x y rpy_r rpy_p rpy_y">
-    <link name="${name}">
-      <visual>
-        <geometry>
-          <mesh filename="package://omnibot_description/meshes/wheel.stl" scale="1 1 1"/>
-        </geometry>
-        <!-- Z = H_wheel/2 -->
-        <origin xyz="0 0 0.04" rpy="0 0 0"/>
-        <material name="black">
-          <color rgba="0.02 0.02 0.02 1"/>
-        </material>
-      </visual>
-      <collision>
-        <geometry>
-          <mesh filename="package://omnibot_description/meshes/wheel.stl" scale="1 1 1"/>
-        </geometry>
-        <origin xyz="0 0 0.04" rpy="0 0 0"/>
-      </collision>
-      <inertial>
-        <mass value="0.2"/>
-        <inertia ixx="0.001" iyy="0.001" izz="0.001" ixy="0" ixz="0" iyz="0"/>
-      </inertial>
-    </link>
-    <joint name="${name}_joint" type="continuous">
-      <parent link="base_link"/>
-      <child link="${name}"/>
-      <!-- Position relativ zum base_link -->
-      <origin xyz="${x} ${y} 0" rpy="${rpy_r} ${rpy_p} ${rpy_y}"/>
-      <axis xyz="0 1 0"/>
-    </joint>
-  </xacro:macro>
   <!-- ================= Four Mecanum Wheels ================= -->
-  <xacro:wheel name="wheel_fl" x="0.12" y="0.12" rpy_r="0" rpy_p="0" rpy_y="0"/>
-  <xacro:wheel name="wheel_fr" x="0.12" y="-0.12" rpy_r="0" rpy_p="0" rpy_y="0"/>
-  <xacro:wheel name="wheel_rl" x="-0.12" y="0.12" rpy_r="0" rpy_p="0" rpy_y="0"/>
-  <xacro:wheel name="wheel_rr" x="-0.12" y="-0.12" rpy_r="0" rpy_p="0" rpy_y="0"/>
+  <!-- Front Left Wheel -->
+  <link name="wheel_fl">
+    <visual>
+      <geometry>
+        <mesh filename="package://omnibot_description/meshes/wheel_fl.stl" scale="1 1 1"/>
+      </geometry>
+      <origin xyz="-0.088 0.100 0.0" rpy="0 0 0"/>
+      <material name="black">
+        <color rgba="0.02 0.02 0.02 1"/>
+      </material>
+    </visual>
+    <collision>
+      <geometry>
+        <mesh filename="package://omnibot_description/meshes/wheel_fl.stl" scale="1 1 1"/>
+      </geometry>
+      <origin xyz="0 0 0" rpy="0 0 0"/>
+    </collision>
+    <inertial>
+      <mass value="0.2"/>
+      <inertia ixx="0.001" iyy="0.001" izz="0.001" ixy="0" ixz="0" iyz="0"/>
+    </inertial>
+  </link>
+  <joint name="wheel_fl_joint" type="continuous">
+    <parent link="base_link"/>
+    <child link="wheel_fl"/>
+    <origin xyz="0.088 -0.100 0.0" rpy="0 0 0"/>
+    <axis xyz="0 1 0"/>
+  </joint>
+  <!-- Front Right Wheel -->
+  <link name="wheel_fr">
+    <visual>
+      <geometry>
+        <mesh filename="package://omnibot_description/meshes/wheel_fr.stl" scale="1 1 1"/>
+      </geometry>
+      <origin xyz="-0.088 0.100 0.0" rpy="0 0 0"/>
+      <material name="black">
+        <color rgba="0.02 0.02 0.02 1"/>
+      </material>
+    </visual>
+    <collision>
+      <geometry>
+        <mesh filename="package://omnibot_description/meshes/wheel_fr.stl" scale="1 1 1"/>
+      </geometry>
+      <origin xyz="0 0 0" rpy="0 0 0"/>
+    </collision>
+    <inertial>
+      <mass value="0.2"/>
+      <inertia ixx="0.001" iyy="0.001" izz="0.001" ixy="0" ixz="0" iyz="0"/>
+    </inertial>
+  </link>
+  <joint name="wheel_fr_joint" type="continuous">
+    <parent link="base_link"/>
+    <child link="wheel_fr"/>
+    <origin xyz="0.088 -0.100 0.0" rpy="0 0 0"/>
+    <axis xyz="0 1 0"/>
+  </joint>
+  <!-- Rear Left Wheel -->
+  <link name="wheel_rl">
+    <visual>
+      <geometry>
+        <mesh filename="package://omnibot_description/meshes/wheel_rl.stl" scale="1 1 1"/>
+      </geometry>
+      <origin xyz="0.103 -0.100 0" rpy="0 0 0"/>
+      <material name="black">
+        <color rgba="0.02 0.02 0.02 1"/>
+      </material>
+    </visual>
+    <collision>
+      <geometry>
+        <mesh filename="package://omnibot_description/meshes/wheel_rl.stl" scale="1 1 1"/>
+      </geometry>
+      <origin xyz="0 0 0" rpy="0 0 0"/>
+    </collision>
+    <inertial>
+      <mass value="0.2"/>
+      <inertia ixx="0.001" iyy="0.001" izz="0.001" ixy="0" ixz="0" iyz="0"/>
+    </inertial>
+  </link>
+  <joint name="wheel_rl_joint" type="continuous">
+    <parent link="base_link"/>
+    <child link="wheel_rl"/>
+    <origin xyz="-0.103 0.100 0" rpy="0 0 0"/>
+    <axis xyz="0 1 0"/>
+  </joint>
+  <!-- Rear Right Wheel -->
+  <link name="wheel_rr">
+    <visual>
+      <geometry>
+        <mesh filename="package://omnibot_description/meshes/wheel_rr.stl" scale="1 1 1"/>
+      </geometry>
+      <origin xyz="0.103 -0.100 0" rpy="0 0 0"/>
+      <material name="black">
+        <color rgba="0.02 0.02 0.02 1"/>
+      </material>
+    </visual>
+    <collision>
+      <geometry>
+        <mesh filename="package://omnibot_description/meshes/wheel_rr.stl" scale="1 1 1"/>
+      </geometry>
+      <origin xyz="0 0 0" rpy="0 0 0"/>
+    </collision>
+    <inertial>
+      <mass value="0.2"/>
+      <inertia ixx="0.001" iyy="0.001" izz="0.001" ixy="0" ixz="0" iyz="0"/>
+    </inertial>
+  </link>
+  <joint name="wheel_rr_joint" type="continuous">
+    <parent link="base_link"/>
+    <child link="wheel_rr"/>
+    <origin xyz="-0.103 0.100 0" rpy="0 0 0"/>
+    <axis xyz="0 1 0"/>
+  </joint>
 </robot>

Commit message: FIx: TFs Wheels

File: urdf/omnibot.urdf.xacro (robot description, xacro)
@@ -30,5 +30,5 @@
         <mesh filename="package://omnibot_description/meshes/wheel_fl.stl" scale="1 1 1"/>
       </geometry>
-      <origin xyz="-0.088 0.100 0.0" rpy="0 0 0"/>
+      <origin xyz="-0.088 -0.100 0.0" rpy="0 0 0"/>
       <material name="black">
         <color rgba="0.02 0.02 0.02 1"/>
@@ -49,5 +49,5 @@
     <parent link="base_link"/>
     <child link="wheel_fl"/>
-    <origin xyz="0.088 -0.100 0.0" rpy="0 0 0"/>
+    <origin xyz="0.088 0.100 0.0" rpy="0 0 0"/>
     <axis xyz="0 1 0"/>
   </joint>
@@ -114,5 +114,5 @@
         <mesh filename="package://omnibot_description/meshes/wheel_rr.stl" scale="1 1 1"/>
       </geometry>
-      <origin xyz="0.103 -0.100 0" rpy="0 0 0"/>
+      <origin xyz="0.103 0.100 0" rpy="0 0 0"/>
       <material name="black">
         <color rgba="0.02 0.02 0.02 1"/>
@@ -133,5 +133,5 @@
     <parent link="base_link"/>
     <child link="wheel_rr"/>
-    <origin xyz="-0.103 0.100 0" rpy="0 0 0"/>
+    <origin xyz="-0.103 -0.100 0" rpy="0 0 0"/>
     <axis xyz="0 1 0"/>
   </joint>
