Commit message: export ROS_DOMAIN_ID and edit URDF (CHANGE BASE TO BASE_LINK in CAD)

File: urdf/robot.urdf (robot description, URDF)
Before this commit: robot omnibot-onshape, 5 links, 4 joints
Links:
- removed link base
- added link base_link, mass 0.427697; collision mesh filename=package://omnibot_description/assets/base.stl; collision mesh filename=package://omnibot_description/assets/part_2.stl
Joints:
- joint wheel_fl: parent base -> base_link
- joint wheel_fr: parent base -> base_link
- joint wheel_rl: parent base -> base_link
- joint wheel_rr: parent base -> base_link
