Commit message: feat(urdf): replace onshape model with correctly oriented export
New OnShape export with +X-forward ROS-standard frame. Replaces old
generic part meshes with named body meshes (base_link, wheels, plates,
battery, camera, etc.).

File: urdf/robot.urdf (robot description, URDF)
Before this commit: robot edubot-onshape, 5 links, 4 joints
Links:
- link base_link: mass 0.427697 -> 0.421125; geometry collision mesh filename=package://edubot_description/assets/axle.stl; collision mesh filename=package://edubot_description/assets/axle.stl
Joints:
- joint wheel_fl: origin xyz=0.0924914 -0.087 0.0185 rpy=-0 -1.5708 0 -> xyz=0.0874013 0.0924166 0.0196934 rpy=1.5708 -1.53297 -0
- joint wheel_fr: origin xyz=-0.0897148 -0.086999 0.0184759 rpy=-3.14159 -1.5708 0 -> xyz=0.087399 -0.0897897 0.0184759 rpy=-1.5708 -1.5708 0
- joint wheel_rl: origin xyz=0.0897148 0.086999 0.0184759 rpy=-1.5708 -0 1.5708 -> xyz=-0.086599 0.0896399 0.0184759 rpy=-1.5708 -0 -3.14159
- joint wheel_rr: origin xyz=-0.0897148 0.087001 0.0184759 rpy=1.5708 -0 1.5708 -> xyz=-0.086601 -0.0897897 0.0184759 rpy=1.5708 -0 -3.14159

Commit message: fix(urdf): flip joint axis for left wheels to match physical orientation

File: urdf/robot.urdf (robot description, URDF)
Before this commit: robot omnibot-onshape, 5 links, 4 joints
Joints:
- joint wheel_fl: axis 0 0 1 -> 0 0 -1
- joint wheel_rl: axis 0 0 1 -> 0 0 -1

Commit message: feat(urdf): add imu_link fixed joint for BNO085

File: urdf/robot.urdf (robot description, URDF)
Before this commit: robot edubot-onshape, 5 links, 4 joints
Links:
- added link imu_link
Joints:
- added joint imu_joint: type fixed, parent base_link, child imu_link, origin xyz=0.0 0.0 0.065 rpy=0 0 0
