Commit message: refactor: rename omnibot to edubot across the repo

File: urdf/edubot.urdf.xacro (robot description, xacro)
@@ -1,9 +1,9 @@
 <?xml version="1.0"?>
-<robot xmlns:xacro="http://www.ros.org/wiki/xacro" name="omnibot">
+<robot xmlns:xacro="http://www.ros.org/wiki/xacro" name="edubot">
   <!-- ================= Base Link ================= -->
   <link name="base_link">
     <visual>
       <geometry>
-        <mesh filename="package://omnibot_description/meshes/base.stl" scale="1 1 1"/>
+        <mesh filename="package://edubot_description/meshes/base.stl" scale="1 1 1"/>
       </geometry>
       <origin xyz="0 0 0" rpy="0 0 0"/>
@@ -14,5 +14,5 @@
     <collision>
       <geometry>
-        <mesh filename="package://omnibot_description/meshes/base.stl" scale="1 1 1"/>
+        <mesh filename="package://edubot_description/meshes/base.stl" scale="1 1 1"/>
       </geometry>
       <origin xyz="0 0 0" rpy="0 0 0"/>
@@ -28,5 +28,5 @@
     <visual>
       <geometry>
-        <mesh filename="package://omnibot_description/meshes/wheel_fl.stl" scale="1 1 1"/>
+        <mesh filename="package://edubot_description/meshes/wheel_fl.stl" scale="1 1 1"/>
       </geometry>
       <origin xyz="-0.088 -0.100 0.0" rpy="0 0 0"/>
@@ -37,5 +37,5 @@
     <collision>
       <geometry>
-        <mesh filename="package://omnibot_description/meshes/wheel_fl.stl" scale="1 1 1"/>
+        <mesh filename="package://edubot_description/meshes/wheel_fl.stl" scale="1 1 1"/>
       </geometry>
       <origin xyz="0 0 0" rpy="0 0 0"/>
@@ -56,5 +56,5 @@
     <visual>
       <geometry>
-        <mesh filename="package://omnibot_description/meshes/wheel_fr.stl" scale="1 1 1"/>
+        <mesh filename="package://edubot_description/meshes/wheel_fr.stl" scale="1 1 1"/>
       </geometry>
       <origin xyz="-0.088 0.100 0.0" rpy="0 0 0"/>
@@ -65,5 +65,5 @@
     <collision>
       <geometry>
-        <mesh filename="package://omnibot_description/meshes/wheel_fr.stl" scale="1 1 1"/>
+        <mesh filename="package://edubot_description/meshes/wheel_fr.stl" scale="1 1 1"/>
       </geometry>
       <origin xyz="0 0 0" rpy="0 0 0"/>
@@ -84,5 +84,5 @@
     <visual>
       <geometry>
-        <mesh filename="package://omnibot_description/meshes/wheel_rl.stl" scale="1 1 1"/>
+        <mesh filename="package://edubot_description/meshes/wheel_rl.stl" scale="1 1 1"/>
       </geometry>
       <origin xyz="0.103 -0.100 0" rpy="0 0 0"/>
@@ -93,5 +93,5 @@
     <collision>
       <geometry>
-        <mesh filename="package://omnibot_description/meshes/wheel_rl.stl" scale="1 1 1"/>
+        <mesh filename="package://edubot_description/meshes/wheel_rl.stl" scale="1 1 1"/>
       </geometry>
       <origin xyz="0 0 0" rpy="0 0 0"/>
@@ -112,5 +112,5 @@
     <visual>
       <geometry>
-        <mesh filename="package://omnibot_description/meshes/wheel_rr.stl" scale="1 1 1"/>
+        <mesh filename="package://edubot_description/meshes/wheel_rr.stl" scale="1 1 1"/>
       </geometry>
       <origin xyz="0.103 0.100 0" rpy="0 0 0"/>
@@ -121,5 +121,5 @@
     <collision>
       <geometry>
-        <mesh filename="package://omnibot_description/meshes/wheel_rr.stl" scale="1 1 1"/>
+        <mesh filename="package://edubot_description/meshes/wheel_rr.stl" scale="1 1 1"/>
       </geometry>
       <origin xyz="0 0 0" rpy="0 0 0"/>

File: urdf/robot.urdf (robot description, URDF)
Before this commit: robot omnibot-onshape, 5 links, 4 joints
Links:
- link base_link: geometry collision mesh filename=package://edubot_description/assets/base.stl; collision mesh filename=package://edubot_description/assets/part_2.stl
- link omni_wheel_fl: geometry collision mesh filename=package://edubot_description/assets/omni_wheel_fl.stl; visual mesh filename=package://edubot_description/assets/omni_wheel_fl.stl
- link omni_wheel_fr: geometry collision mesh filename=package://edubot_description/assets/omni_wheel_fr.stl; visual mesh filename=package://edubot_description/assets/omni_wheel_fr.stl
- link omni_wheel_rl: geometry collision mesh filename=package://edubot_description/assets/omni_wheel_rl.stl; visual mesh filename=package://edubot_description/assets/omni_wheel_rl.stl
- link omni_wheel_rr: geometry collision mesh filename=package://edubot_description/assets/omni_wheel_rr.stl; visual mesh filename=package://edubot_description/assets/omni_wheel_rr.stl
